Commit message: Custom robot structure

File: husky_description/urdf/custom_description.urdf.xacro (robot description, xacro)
@@ -21,17 +21,17 @@
 ARISING IN ANY WAY OUT OF THE USE OF THIS SOFTWARE, EVEN IF ADVISED OF THE POSSIBILITY OF SUCH DAMAGE.
 -->
-<robot name="husky" xmlns:xacro="http://ros.org/wiki/xacro">
+<robot name="husky_robot" xmlns:xacro="http://ros.org/wiki/xacro">
   <xacro:arg name="laser_enabled" default="$(optenv HUSKY_LMS1XX_ENABLED false)" />
   <xacro:arg name="ur5_enabled" default="$(optenv HUSKY_UR5_ENABLED false)" />
   <xacro:arg name="kinect_enabled" default="false" />
+  <xacro:arg name="hesai_lidar_enabled" default="true" />
   <xacro:include filename="$(find husky_description)/urdf/husky.urdf.xacro" />
-  <xacro:husky_robot />
-<!--- Insert Customizations Below -->
-<!-- Sensor arch with GPS and Axis Camera -->
+  <!-- Insert customization below: sample provided  -->
+  <!-- Sensor arch with GPS and Axis Camera -->
   <link name="sensorArch">
    <visual>
     <origin xyz="-0.08 0 0.007" rpy="0 0 0"/>
     <geometry>
-    <mesh filename="package://husky_custom_description/meshes/sensorArch.dae" />
+    <mesh filename="package://husky_description/meshes/custom/sensorArch.dae" />
     </geometry>
    </visual>
@@ -41,10 +41,10 @@
     <child link="sensorArch" />
   </joint>
-<!-- Quanergy M8 on the Left -->
-  <link name="sensor_left">
+  <!-- Quanergy M8 on the Left -->
+  <!--link name="sensor_left">
    <visual>
     <origin xyz="0 0 0" rpy="0 0 1.5708" />
     <geometry>
-    <mesh filename="package://husky_custom_description/meshes/quanergyM8.dae" />
+    <mesh filename="package://husky_description/meshes/custom/quanergyM8.dae" />
     </geometry>
    </visual>
@@ -54,11 +54,11 @@
     <child link="sensor_left" />
     <origin xyz="-0.08 0.285 0.583"  rpy="-0.785398 0 0" />
-  </joint>
-<!-- Quanergy M8 on the Right -->
-  <link name="sensor_right">
+  </joint-->
+  <!-- Quanergy M8 on the Right -->
+  <!--link name="sensor_right">
    <visual>
     <origin xyz="0 0 0" rpy="0 0 1.5708" />
     <geometry>
-    <mesh filename="package://husky_custom_description/meshes/quanergyM8.dae" />
+    <mesh filename="package://husky_description/meshes/custom/quanergyM8.dae" />
     </geometry>
    </visual>
@@ -68,11 +68,11 @@
     <child link="sensor_right" />
     <origin xyz="-0.08 -0.286 0.583" rpy="0.785398 0 0"/>
-  </joint>
-<!-- Hesai Pandar 40 Lidar -->
-  <link name="sensor_hesai">
+  </joint-->
+  <!-- Hesai Pandar 40 Lidar -->
+  <!--link name="sensor_hesai">
    <visual>
     <origin xyz="0 0 -0.032" rpy="0 0 0" />
     <geometry>
-    <mesh filename="package://husky_custom_description/meshes/hesaiLiDAR.dae" />
+    <mesh filename="package://husky_description/meshes/custom/hesaiLiDAR.dae" />
     </geometry>
    </visual>
@@ -82,11 +82,34 @@
     <child link="sensor_hesai" />
     <origin xyz="-0.08 0 0.695" rpy="0 0 1.5708"/>
-  </joint>
-<!-- LMS151 Front Lidar -->
+  </joint-->
+  <!-- simplified lidar for quick launch-->
+  <xacro:macro name="velodyne_lidar">
+    <xacro:property name="M_PI" value="3.1415926535897931" />
+    <xacro:include filename="$(find velodyne_description)/urdf/VLP-16.urdf.xacro"/>
+  <VLP-16 parent="top_plate_link"
+              name="velodyne"
+              topic="/velodyne_points"
+              hz="8"
+              samples="1100"
+              lasers="36"
+              collision_range ="0.3"
+              min_range ="0.3"
+              max_range ="200.0"
+              noise ="0.1"
+              min_angle_hor="-${M_PI}"
+              max_angle_hor="${M_PI}"
+              min_angle_ver="-16"
+              max_angle_ver="7"
+              >
+      <origin xyz="-0.08 0 0.695" rpy="0 0 0" />
+  </VLP-16>
+  </xacro:macro>
+  <xacro:velodyne_lidar />
+  <!-- LMS151 Front Lidar -->
   <link name="laser">
    <visual>
     <origin xyz="0 0 0" rpy="3.1415 0 -1.5708" />
     <geometry>
-    <mesh filename="package://husky_custom_description/meshes/lms151.dae" />
+    <mesh filename="package://husky_description/meshes/custom/lms151.dae" />
     </geometry>
    </visual>
@@ -97,3 +120,4 @@
     <origin xyz="0.3 0 0" rpy="3.1415 0 0"/>
   </joint>
+  <xacro:husky_robot />
 </robot>

File: husky_gazebo/urdf/description.gazebo.xacro (robot description, xacro)
@@ -34,5 +34,5 @@
   </gazebo>
   <!--<xacro:husky_robot />-->
-  <xacro:include filename="$(find husky_description)/urdf/my_description.urdf.xacro" />
+  <xacro:include filename="$(find husky_description)/urdf/custom_description.urdf.xacro" />
   <xacro:husky_robot_gazebo />
   <!-- Insert customizations below: -->

Commit message: modify the visilization of robot model in gazebo environment, note that the husky_viz need more modification

File: husky_description/urdf/custom_description.urdf.xacro (robot description, xacro)
@@ -84,26 +84,8 @@
   </joint-->
   <!-- simplified lidar for quick launch-->
-  <xacro:macro name="velodyne_lidar">
-    <xacro:property name="M_PI" value="3.1415926535897931" />
-    <xacro:include filename="$(find velodyne_description)/urdf/VLP-16.urdf.xacro"/>
-  <VLP-16 parent="top_plate_link"
-              name="velodyne"
-              topic="/velodyne_points"
-              hz="10"
-              samples="1100"
-              lasers="16"
-              collision_range ="0.3"
-              min_range ="0.3"
-              max_range ="200.0"
-              noise ="0.01"
-              min_angle_hor="-${M_PI}"
-              max_angle_hor="${M_PI}"
-              min_angle_ver="-15"
-              max_angle_ver="15"
-              >
-      <origin xyz="-0.08 0 0.695" rpy="0 0 0" />
+  <xacro:include filename="$(find velodyne_description)/urdf/VLP-16.urdf.xacro"/>
+  <VLP-16 parent="sensorArch" name="velodyne_lidar" topic="/velodyne_points">
+    <origin xyz="-0.08 0 0.15" rpy="0 0 0" />
   </VLP-16>
-  </xacro:macro>
-  <xacro:velodyne_lidar />
   <!-- LMS151 Front Lidar -->
   <link name="laser">

File: velodyne_description/urdf/VLP-16-raw.urdf.xacro (robot description, xacro)
@@ -27,4 +27,14 @@
         <inertia ixx="0.1" ixy="0" ixz="0" iyy="0.1" iyz="0" izz="0.1"/>
       </inertial>
+      <visual>
+        <geometry>
+          <mesh filename="package://velodyne_description/meshes/VLP16_base_1.dae" />
+        </geometry>
+      </visual>
+      <visual>
+        <geometry>
+          <mesh filename="package://velodyne_description/meshes/VLP16_base_2.dae" />
+        </geometry>
+      </visual>
       <collision>
         <origin rpy="0 0 0" xyz="0 0 0.03585"/>
@@ -45,10 +55,10 @@
         <inertia ixx="0.1" ixy="0" ixz="0" iyy="0.1" iyz="0" izz="0.1"/>
       </inertial>
-      <!--visual>
+      <visual>
         <origin xyz="0 0 -0.0377" />
         <geometry>
           <mesh filename="package://velodyne_description/meshes/VLP16_scan.dae" />
         </geometry>
-      </visual-->
+      </visual>
     </link>
     <!-- Gazebo requires the velodyne_gazebo_plugins package -->
